File: Comp1.kicad_sch (KiCad schematic)
At the start: 12 parts, among them U4 LM431BIM3/NOPB, U5 SFH615A-3X009

Commit message: 完善补偿电路原理图；
Parts:
- added R43, R52: 0, Resistor_SMD:R_0603_1608Metric_Pad0.98x0.95mm_HandSolder, symbol Device:R_Small_US
- added R51: 5.1k, Resistor_SMD:R_0603_1608Metric_Pad0.98x0.95mm_HandSolder, symbol Device:R_Small_US
- added Rz1: 0, Resistor_SMD:R_1206_3216Metric_Pad1.30x1.75mm_HandSolder, symbol Device:R_Small_US
- renumbered RBode to RBode1, Rled to Rled1
Connections:
- net GND1: now also R43.1; no longer R41.1
- net at R39.2, RBode1.1: now also Rz1.1; no longer Rled1.2
- net Vdiv: now reaches C50.1, R41.2, R44.1, R45.1, U4.2 (Reference)
- net at U5.4 (COL): now also R51.2, R52.1
- net VOUT renamed Vout
- new net: Rled1.2, Rz1.2
- new net: R41.1, R43.2
- new net 5V_PullUp: R51.1
- new net FB1: R52.2
Other:
- moved on the sheet: Rled1

Commit message: 初版布局连线；
Parts:
- added TP12: Bode, TestPoint:TestPoint_Keystone_5005-5009_Compact, symbol Connector:TestPoint
Connections:
- net at R39.2, RBode1.1, Rz1.1: now also TP12.1
