File: Start Up.kicad_sch (KiCad schematic)
At the start: 14 parts, among them Q2 MMBT3904, Q3 BSP129, U6 TLV70450DBVR

Commit message: 初版布局连线；
Parts:
- added C36: 100n, Capacitor_SMD:C_0603_1608Metric_Pad1.08x0.95mm_HandSolder, symbol Device:C
- added C67: 120p, Capacitor_SMD:C_0603_1608Metric_Pad1.08x0.95mm_HandSolder, symbol Device:C
- added R33: 1.5k, Resistor_SMD:R_0603_1608Metric_Pad0.98x0.95mm_HandSolder, symbol Device:R_Small_US
- added R64: 100k, Resistor_SMD:R_1206_3216Metric_Pad1.30x1.75mm_HandSolder, symbol Device:R_Small_US
- added R65: 5.1k, Resistor_SMD:R_0805_2012Metric_Pad1.20x1.40mm_HandSolder, symbol Device:R_Small_US
Connections:
- net GND: now also C36.1, C67.1, R65.2
- net VIN: now also R64.1
- net at Q2.1 (B), R31.2, R32.2: now also C36.2
- net 5V_LDO: now reaches C35.2, U6.3 (OUT)
- new net OP1-: C67.2, R33.2, R64.2, R65.1
- new net OP1o/Ramp: R33.1
