File: FlyBack_pic16f1769.kicad_pcb (KiCad board)
At the start: 2 copper layers, 100 x 100 mm, 102 parts, among them J1 ICSP, Q1 IPD50R380CE, T1 Transformer_PQ2020A_6+8, U1 PIC16F1769-I/P, U2 MCP1416, U3 ADUM3190ARQZ-RL7, U4 LM431BIM3/NOPB, U5 SFH615A-3X009

Commit message: 完善补偿电路原理图；
Parts:
- removed C10, C20, C27, C34, C41, C42: 10u, Capacitor_SMD:CP_Elec_10x12.5
- added C49: 47n, Capacitor_SMD:C_0603_1608Metric_Pad1.08x0.95mm_HandSolder, F.Cu at (101.6, 123.1)
- added C50: 10n, Capacitor_SMD:C_0603_1608Metric_Pad1.08x0.95mm_HandSolder, F.Cu at (101.6, 125.6)
- added C51: 10n, Capacitor_SMD:C_0603_1608Metric_Pad1.08x0.95mm_HandSolder, F.Cu at (75.6, 149.2)
- added C52: 47n, Capacitor_SMD:C_0603_1608Metric_Pad1.08x0.95mm_HandSolder, F.Cu at (75.6, 151.7)
- added C53: 100n, Capacitor_SMD:C_0603_1608Metric_Pad1.08x0.95mm_HandSolder, F.Cu at (75.6, 154.2)
- added C54: 100n, Capacitor_SMD:C_0603_1608Metric_Pad1.08x0.95mm_HandSolder, F.Cu at (75.6, 156.7)
- added C55: 1u, Capacitor_SMD:C_0603_1608Metric_Pad1.08x0.95mm_HandSolder, F.Cu at (75.6, 159.3)
- added C56: 1u, Capacitor_SMD:C_0603_1608Metric_Pad1.08x0.95mm_HandSolder, F.Cu at (79.9, 149.2)
- added C57: 1u, Capacitor_SMD:C_0603_1608Metric_Pad1.08x0.95mm_HandSolder, F.Cu at (79.9, 151.7)
- added C58: 1u, Capacitor_SMD:C_0603_1608Metric_Pad1.08x0.95mm_HandSolder, F.Cu at (79.9, 154.2)
- added C59: 15p, Capacitor_SMD:C_0603_1608Metric_Pad1.08x0.95mm_HandSolder, F.Cu at (79.9, 156.7)
- added C60: 15p, Capacitor_SMD:C_0603_1608Metric_Pad1.08x0.95mm_HandSolder, F.Cu at (79.9, 159.3)
- added C61: 10u, Capacitor_SMD:C_1206_3216Metric_Pad1.33x1.80mm_HandSolder, F.Cu at (29.0, 98.3)
- added C62: 10u, Capacitor_SMD:C_1206_3216Metric_Pad1.33x1.80mm_HandSolder, F.Cu at (29.0, 101.7)
- added C63: 10u, Capacitor_SMD:C_1206_3216Metric_Pad1.33x1.80mm_HandSolder, F.Cu at (29.0, 105.0)
- added C64: 100n, Capacitor_SMD:C_0603_1608Metric_Pad1.08x0.95mm_HandSolder, F.Cu at (33.3, 87.8)
- added C66: 10u, Capacitor_SMD:CP_Elec_10x12.5, F.Cu at (18.9, 104.6)
- added D8: D, Diode_SMD:D_SMC, F.Cu at (34.6, 113.0)
- added R39: 1k, Resistor_SMD:R_0603_1608Metric_Pad0.98x0.95mm_HandSolder, F.Cu at (101.6, 128.1)
- added R40: 3.9k, Resistor_SMD:R_0603_1608Metric_Pad0.98x0.95mm_HandSolder, F.Cu at (101.6, 130.6)
- added R41: 1.47k, Resistor_SMD:R_0603_1608Metric_Pad0.98x0.95mm_HandSolder, F.Cu at (101.6, 133.2)
- added R42: NC, Resistor_SMD:R_0603_1608Metric_Pad0.98x0.95mm_HandSolder, F.Cu at (101.6, 135.7)
- added R43: 0, Resistor_SMD:R_0603_1608Metric_Pad0.98x0.95mm_HandSolder, F.Cu at (101.6, 138.2)
- added R44: 4.7k, Resistor_SMD:R_0603_1608Metric_Pad0.98x0.95mm_HandSolder, F.Cu at (101.6, 140.7)
- added R45: 0, Resistor_SMD:R_0603_1608Metric_Pad0.98x0.95mm_HandSolder, F.Cu at (101.6, 143.2)
- added R46: 4.7k, Resistor_SMD:R_0603_1608Metric_Pad0.98x0.95mm_HandSolder, F.Cu at (84.3, 149.2)
- added R47: 0, Resistor_SMD:R_0603_1608Metric_Pad0.98x0.95mm_HandSolder, F.Cu at (84.3, 151.7)
- added R48: 10, Resistor_SMD:R_1206_3216Metric_Pad1.30x1.75mm_HandSolder, F.Cu at (91.0, 143.7)
- added R49: 10k, Resistor_SMD:R_0603_1608Metric_Pad0.98x0.95mm_HandSolder, F.Cu at (84.3, 154.2)
- added R50: 0, Resistor_SMD:R_0603_1608Metric_Pad0.98x0.95mm_HandSolder, F.Cu at (84.3, 156.7)
- added R51: 5.1k, Resistor_SMD:R_0603_1608Metric_Pad0.98x0.95mm_HandSolder, F.Cu at (147.6, 110.2)
- added R52: 0, Resistor_SMD:R_0603_1608Metric_Pad0.98x0.95mm_HandSolder, F.Cu at (147.6, 112.7)
- added RBode1: 10, Resistor_SMD:R_1206_3216Metric_Pad1.30x1.75mm_HandSolder, F.Cu at (106.7, 123.5)
- added Rled1: 2.4k, Resistor_SMD:R_1206_3216Metric_Pad1.30x1.75mm_HandSolder, F.Cu at (106.7, 126.8)
- added Rz1: 0, Resistor_SMD:R_1206_3216Metric_Pad1.30x1.75mm_HandSolder, F.Cu at (106.7, 130.1)
- added TP1: Vout, TestPoint:TestPoint_Keystone_5005-5009_Compact, F.Cu at (90.5, 124.4)
- added TP2: Vin, TestPoint:TestPoint_Keystone_5005-5009_Compact, F.Cu at (28.6, 94.1)
- added TP3: VFB, TestPoint:TestPoint_Keystone_5005-5009_Compact, F.Cu at (140.9, 111.5)
Connections:
- C13 pad 2: Net-(D1-K) -> /Vout
- C14 pad 2: Net-(D1-K) -> /Vout
- C15 pad 2: Net-(D1-K) -> /Vout
- C8 pad 2: Net-(D1-K) -> /Vout
- C9 pad 1: Net-(D1-K) -> /Vout
- D1 pad 1: Net-(D1-K) -> /Vout
- R17 pad 2: Net-(D1-K) -> /Vout
- R18 pad 2: Net-(D1-K) -> /Vout
- R8 pad 2: Net-(D1-K) -> /Vout
- R9 pad 2: Net-(D1-K) -> /Vout
- U3 pad 1: unconnected-(U3-VDD1-Pad1) -> /Comp2/VDD1
- U3 pad 10: unconnected-(U3-COMP-Pad10) -> Net-(U3-COMP)
- U3 pad 11: unconnected-(U3-IN--Pad11) -> /Comp1/Vdiv
- U3 pad 12: unconnected-(U3-IN+-Pad12) -> Net-(U3-IN+)
- U3 pad 13: unconnected-(U3-REFOUT-Pad13) -> /Comp2/ISO_REFOUT
- U3 pad 14: unconnected-(U3-VREG2-Pad14) -> Net-(U3-VREG2)
- U3 pad 15: unconnected-(U3-GND2-Pad15) -> Net-(C53-Pad1)
- U3 pad 16: unconnected-(U3-VDD2-Pad16) -> /Vout
- U3 pad 2: unconnected-(U3-GND1-Pad2) -> Net-(C54-Pad1)
- U3 pad 3: unconnected-(U3-VREG1-Pad3) -> Net-(U3-VREG1)
- U3 pad 4: unconnected-(U3-REFOUT1-Pad4) -> Net-(U3-REFOUT1)
- U3 pad 5: unconnected-(U3-NC-Pad5) -> GND
- U3 pad 6: unconnected-(U3-EAOUT2-Pad6) -> /Comp2/EAOUT2
- U3 pad 7: unconnected-(U3-EAOUT-Pad7) -> /Comp2/EAOUT
- U3 pad 8: unconnected-(U3-GND1-Pad8) -> GND
- U3 pad 9: unconnected-(U3-GND2-Pad9) -> GND1
- U4 pad 1: unconnected-(U4-Cathode-Pad1) -> Net-(U4-Cathode)
- U4 pad 2: unconnected-(U4-Reference-Pad2) -> /Comp1/Vdiv
- U4 pad 3: unconnected-(U4-Anode-Pad3) -> GND1
- U5 pad 1: unconnected-(U5-AN-Pad1) -> Net-(U5-AN)
- U5 pad 2: unconnected-(U5-CAT-Pad2) -> Net-(U4-Cathode)
- U5 pad 3: unconnected-(U5-EM-Pad3) -> GND
- U5 pad 4: unconnected-(U5-COL-Pad4) -> Net-(U5-COL)

Commit message: 完善启动电路；
Parts:
- removed C35: 220p, Capacitor_SMD:C_1206_3216Metric_Pad1.33x1.80mm_HandSolder
- removed C36, C37, C38: 10u, Capacitor_SMD:C_1206_3216Metric_Pad1.33x1.80mm_HandSolder
- removed C39: 100n, Capacitor_SMD:C_0603_1608Metric_Pad1.08x0.95mm_HandSolder
- removed C40: 10u, Capacitor_SMD:CP_Elec_10x12.5
- removed D6: D, Diode_SMD:D_SMB_Handsoldering
- removed R31, R32: 100, Resistor_SMD:R_1206_3216Metric_Pad1.30x1.75mm_HandSolder
- removed R33, R34: 10k, Resistor_SMD:R_1206_3216Metric_Pad1.30x1.75mm_HandSolder
- added C20: 10u, Capacitor_SMD:C_1206_3216Metric_Pad1.33x1.80mm_HandSolder, F.Cu at (213.3, 48.5)
- added C27: 10u, Capacitor_SMD:C_1206_3216Metric_Pad1.33x1.80mm_HandSolder, F.Cu at (213.3, 51.8)
- added C34: 10u, Capacitor_SMD:C_1206_3216Metric_Pad1.33x1.80mm_HandSolder, F.Cu at (213.3, 55.2)
- added C41: 10u, Capacitor_SMD:C_1206_3216Metric_Pad1.33x1.80mm_HandSolder, F.Cu at (213.3, 58.5)
- added C65: 10u, Capacitor_SMD:C_1206_3216Metric_Pad1.33x1.80mm_HandSolder, F.Cu at (217.1, 121.8)
- added CN1: 640445-3, kicad_api_lib:640445-3, F.Cu at (145.4, 58.4)
- added CN2: 640445-2, kicad_api_lib:640445-2, F.Cu at (344.7, 62.5)
- added CN3: 640445-3, kicad_api_lib:640445-3, F.Cu at (234.5, 14.3)
- added CN4: 640445-3, kicad_api_lib:640445-3, F.Cu at (234.5, 23.6)
- added CN5: 640445-2, kicad_api_lib:640445-2, F.Cu at (344.7, 71.7)
- added D10: MMSZ5226BT1G, kicad_api_lib:MMSZ5226BT1G, F.Cu at (210.8, 129.4)
- added D11: MMSZ5226BT1G, kicad_api_lib:MMSZ5226BT1G, F.Cu at (213.0, 62.1)
- added D9: Z1SMAxxx, Diode_SMD:D_SMA, F.Cu at (218.2, 117.9)
- added R53: 2k, Resistor_SMD:R_1206_3216Metric_Pad1.30x1.75mm_HandSolder, F.Cu at (211.1, 117.3)
- added R54: 2k, Resistor_SMD:R_1206_3216Metric_Pad1.30x1.75mm_HandSolder, F.Cu at (211.1, 120.6)
- added R55: 2k, Resistor_SMD:R_1206_3216Metric_Pad1.30x1.75mm_HandSolder, F.Cu at (211.1, 123.9)
- added R56: 10k, Resistor_SMD:R_1206_3216Metric_Pad1.30x1.75mm_HandSolder, F.Cu at (207.3, 48.5)
- added R57: 10k, Resistor_SMD:R_1206_3216Metric_Pad1.30x1.75mm_HandSolder, F.Cu at (207.3, 51.8)
- added R58: No, Resistor_SMD:R_1206_3216Metric_Pad1.30x1.75mm_HandSolder, F.Cu at (207.3, 55.1)
- added R59: 10k, Resistor_SMD:R_1206_3216Metric_Pad1.30x1.75mm_HandSolder, F.Cu at (207.3, 58.4)
- added R60: 10k, Resistor_SMD:R_1206_3216Metric_Pad1.30x1.75mm_HandSolder, F.Cu at (207.3, 61.7)
- added R61: No, Resistor_SMD:R_1206_3216Metric_Pad1.30x1.75mm_HandSolder, F.Cu at (207.3, 65.0)
- added TP10: Drain, TestPoint:TestPoint_Keystone_5005-5009_Compact, F.Cu at (105.0, 70.5)
- added TP4: Vdrive1, TestPoint:TestPoint_Keystone_5005-5009_Compact, F.Cu at (201.8, 49.3)
- added TP5: GND_drive1, TestPoint:TestPoint_Keystone_5005-5009_Compact, F.Cu at (201.8, 54.4)
- added TP6: Vdrive2, TestPoint:TestPoint_Keystone_5005-5009_Compact, F.Cu at (201.8, 59.4)
- added TP7: GND_drive2, TestPoint:TestPoint_Keystone_5005-5009_Compact, F.Cu at (201.8, 64.5)
- added TP8: Isense, TestPoint:TestPoint_Keystone_5005-5009_Compact, F.Cu at (352.0, 60.4)
- added TP9: GND, TestPoint:TestPoint_Keystone_5005-5009_Compact, F.Cu at (352.0, 65.5)
- moved C26 183.3 mm to (261.2, 58.2)
- moved C29 183.3 mm to (312.6, 41.8)
- moved C30 183.3 mm to (312.6, 45.1)
- moved C31 183.3 mm to (312.6, 48.5)
- moved C45 183.3 mm to (318.6, 41.8)
- moved C46 183.3 mm to (318.6, 45.1)
- moved C47 183.3 mm to (318.6, 48.5)
- moved C48 183.3 mm to (318.6, 51.8)
- moved J1 183.3 mm to (301.9, 89.9)
- moved R24 183.3 mm to (264.6, 77.9)
- moved R25 183.3 mm to (264.6, 81.2)
- moved R26 183.3 mm to (264.6, 84.5)
- moved R27 183.3 mm to (264.6, 87.8)
- moved R28 183.3 mm to (264.6, 91.1)
- moved R29 183.3 mm to (264.6, 94.4)
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Connections:
- net Net-(C12-Pad1) renamed /GND_drive1
- net Net-(C22-Pad1) renamed /GND_drive2
- net Net-(D3-K) renamed /Vdrive1
- net Net-(D4-K) renamed /Vdrive2
- C13 pad 1: Net-(C13-Pad1) -> GND1
- C14 pad 1: Net-(C13-Pad1) -> GND1
- C15 pad 1: Net-(C13-Pad1) -> GND1
- C43 pad 2: Net-(C43-Pad2) -> GND
- C44 pad 1: Net-(C43-Pad2) -> GND
- C45 pad 1: Net-(C43-Pad2) -> GND
- C46 pad 1: Net-(C43-Pad2) -> GND
- C47 pad 1: Net-(C43-Pad2) -> GND
- C54 pad 2: /Comp2/VDD1 -> Vdrive
- C55 pad 2: /Comp2/VDD1 -> Vdrive
- C8 pad 1: Net-(C13-Pad1) -> GND1
- C9 pad 2: Net-(C13-Pad1) -> GND1
- R17 pad 1: Net-(C13-Pad1) -> GND1
- R18 pad 1: Net-(C13-Pad1) -> GND1
- R35 pad 1: Net-(C43-Pad2) -> GND
- R36 pad 1: Net-(C43-Pad2) -> GND
- R49 pad 2: /Comp2/VDD1 -> Vdrive
- T1 pad 3: Net-(D6-A) -> unconnected-(T1-Pad3)
- T1 pad 4: Net-(C36-Pad1) -> unconnected-(T1-Pad4)
- T1 pad 6: Net-(C43-Pad2) -> GND
- T1 pad 8: Net-(C13-Pad1) -> GND1
- U3 pad 1: /Comp2/VDD1 -> Vdrive

Commit message: 初版布局连线；
Parts:
- removed C43: 10u, Capacitor_SMD:CP_Elec_10x12.5
- added C10: 100n, Capacitor_SMD:C_0603_1608Metric_Pad1.08x0.95mm_HandSolder, F.Cu at (74.9, 64.4)
- added C35: 1u, Capacitor_SMD:C_0603_1608Metric_Pad1.08x0.95mm_HandSolder, F.Cu at (77.5, 61.7)
- added C36: 100n, Capacitor_SMD:C_0603_1608Metric_Pad1.08x0.95mm_HandSolder, F.Cu at (106.2, 57.3)
- added C37: 100n, Capacitor_SMD:C_0603_1608Metric_Pad1.08x0.95mm_HandSolder, F.Cu at (57.9, 83.8)
- added C38: 100n, Capacitor_SMD:C_0603_1608Metric_Pad1.08x0.95mm_HandSolder, F.Cu at (57.4, 72.8)
- added C39: 0.47u, Capacitor_SMD:C_0603_1608Metric_Pad1.08x0.95mm_HandSolder, F.Cu at (54.1, 66.5)
- added C40: 1u, Capacitor_SMD:C_0603_1608Metric_Pad1.08x0.95mm_HandSolder, F.Cu at (64.9, 69.1)
- added C67: 120p, Capacitor_SMD:C_0603_1608Metric_Pad1.08x0.95mm_HandSolder, F.Cu at (95.7, 80.8)
- added D6: MBRA340T3G, kicad_api_lib:MBRA340T3G, F.Cu at (74.3, 69.1)
- added J2: TYPE-C-31-M-12, kicad_api_lib:TYPE-C-31-M-12, F.Cu at (60.2, 56.9)
- added Q2: MMBT3904, Package_TO_SOT_SMD:SOT-23, F.Cu at (110.0, 58.2)
- added Q3: BSP129, kicad_api_lib:BSP129, F.Cu at (109.1, 64.5)
- added R31: 10k, Resistor_SMD:R_0603_1608Metric_Pad0.98x0.95mm_HandSolder, F.Cu at (71.9, 67.8)
- added R32: 47k, Resistor_SMD:R_0603_1608Metric_Pad0.98x0.95mm_HandSolder, F.Cu at (106.1, 55.7)
- added R33: 1.5k, Resistor_SMD:R_0603_1608Metric_Pad0.98x0.95mm_HandSolder, F.Cu at (92.2, 80.7)
- added R62: 22k, Resistor_SMD:R_1206_3216Metric_Pad1.30x1.75mm_HandSolder, F.Cu at (102.0, 62.0)
- added R63: 10, Resistor_SMD:R_1206_3216Metric_Pad1.30x1.75mm_HandSolder, F.Cu at (114.8, 63.7)
- added R64: 100k, Resistor_SMD:R_1206_3216Metric_Pad1.30x1.75mm_HandSolder, F.Cu at (114.8, 58.7)
- added R65: 5.1k, Resistor_SMD:R_0805_2012Metric_Pad1.20x1.40mm_HandSolder, F.Cu at (94.0, 80.9)
- added R66: 4.7k, Resistor_SMD:R_0603_1608Metric_Pad0.98x0.95mm_HandSolder, F.Cu at (62.0, 87.5)
- added R67: 4.7k, Resistor_SMD:R_0603_1608Metric_Pad0.98x0.95mm_HandSolder, F.Cu at (60.2, 86.6)
- added R68: 4.7k, Resistor_SMD:R_0603_1608Metric_Pad0.98x0.95mm_HandSolder, F.Cu at (54.2, 72.0)
- added R69: 4.7k, Resistor_SMD:R_0603_1608Metric_Pad0.98x0.95mm_HandSolder, F.Cu at (55.8, 72.0)
- added R70: 5.1k, Resistor_SMD:R_0603_1608Metric_Pad0.98x0.95mm_HandSolder, B.Cu at (61.5, 62.1)
- added R71: 5.1k, Resistor_SMD:R_0603_1608Metric_Pad0.98x0.95mm_HandSolder, B.Cu at (58.5, 62.1)
- added TP11: GND, TestPoint:TestPoint_Keystone_5005-5009_Compact, F.Cu at (76.6, 119.2)
- added TP12: Bode, TestPoint:TestPoint_Keystone_5005-5009_Compact, F.Cu at (63.1, 121.3)
- added TP13: Gate, TestPoint:TestPoint_Keystone_5005-5009_Compact, F.Cu at (115.8, 68.8)
- added U6: TLV70450DBVR, kicad_api_lib:TLV70450DBVR, F.Cu at (75.0, 61.4)
- added U7: MCP2221AxST, Package_SO:TSSOP-14_4.4x5mm_P0.65mm, F.Cu at (59.3, 67.3)
- added U8: ADuM1201BR, Package_SO:SOIC-8_3.9x4.9mm_P1.27mm, F.Cu at (62.8, 78.6)
- added U9: ADuM1250, Package_SO:SOIC-8_3.9x4.9mm_P1.27mm, F.Cu at (56.0, 78.4)
- C19, C26: value 10u -> 100n; footprint Capacitor_SMD:CP_Elec_10x12.5 -> Capacitor_SMD:C_0603_1608Metric_Pad1.08x0.95mm_HandSolder
- R47: footprint Resistor_SMD:R_0603_1608Metric_Pad0.98x0.95mm_HandSolder -> Resistor_SMD:R_0402_1005Metric_Pad0.72x0.64mm_HandSolder
- R53: value 2k -> 22k
- R54: value 2k -> 4.7k; footprint Resistor_SMD:R_1206_3216Metric_Pad1.30x1.75mm_HandSolder -> Resistor_SMD:R_0603_1608Metric_Pad0.98x0.95mm_HandSolder
- R55: value 2k -> 10
- moved CN2 278.7 mm to (74.3, 129.7), turned to 90 degrees
- moved R51 258.1 mm to (72.4, 99.0), turned to -90 degrees
- moved R52 256.5 mm to (74.0, 99.0), turned to 90 degrees
- moved TP9 251.7 mm to (100.9, 83.2)
- moved TP8 251.5 mm to (101.0, 76.4)
- moved TP3 246.4 mm to (77.8, 86.5)
- moved U3 242.8 mm to (61.1, 106.1), turned to -90 degrees
- moved C45 234.4 mm to (89.8, 92.3)
- moved C46 234.2 mm to (89.8, 94.7)
- moved C47 234.0 mm to (89.7, 97.1)
- moved U5 232.2 mm to (75.3, 107.0), turned to 90 degrees
- moved C4 229.6 mm to (79.3, 61.7), turned to -90 degrees
- moved C8 227.3 mm to (85.7, 121.4), turned to -90 degrees
- moved C44 225.9 mm to (89.2, 99.1)
- moved C48 224.3 mm to (99.2, 98.2), turned to -90 degrees
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Connections:
- net /Vin renamed /INPUT
- C19 pad 1: /Vdrive1 -> GND
- C19 pad 2: /GND_drive1 -> +5V
- C26 pad 1: /Vdrive2 -> GNDD
- C26 pad 2: /GND_drive2 -> VDD
- C29 pad 1: Net-(C29-Pad1) -> GND2
- C30 pad 1: Net-(C29-Pad1) -> GND2
- C31 pad 1: Net-(C29-Pad1) -> GND2
- C32 pad 1: Net-(C29-Pad1) -> GND2
- C33 pad 2: Net-(C29-Pad1) -> GND2
- C53 pad 1: Net-(C53-Pad1) -> GND1
- C54 pad 1: Net-(C54-Pad1) -> GND
- C55 pad 1: Net-(C54-Pad1) -> GND
- C56 pad 1: Net-(C53-Pad1) -> GND1
- C57 pad 2: Net-(C54-Pad1) -> GND
- C58 pad 2: Net-(C53-Pad1) -> GND1
- CN5 pad 2: Net-(C29-Pad1) -> GND2
- R29 pad 1: Net-(C29-Pad1) -> GND2
- R30 pad 1: Net-(C29-Pad1) -> GND2
- R48 pad 2: unconnected-(R48-Pad2) -> /Start Up/VAUX
- R53 pad 1: Net-(R53-Pad1) -> Net-(Q2-C)
- R53 pad 2: /P1_1 -> Net-(Q3-GATE)
- R54 pad 1: Net-(R54-Pad1) -> Net-(U7-~{RST})
- R54 pad 2: Net-(R53-Pad1) -> VDD
- R55 pad 1: Vdrive -> Net-(Q3-SOURCE)
- R55 pad 2: Net-(R54-Pad1) -> Vdrive
- T1 pad 13: Net-(D5-A) -> Net-(D1-A)
- T1 pad 14: Net-(C29-Pad1) -> GND1
- T1 pad 7: Net-(D1-A) -> Net-(D5-A)
- T1 pad 8: GND1 -> GND2
- U3 pad 15: Net-(C53-Pad1) -> GND1
- U3 pad 2: Net-(C54-Pad1) -> GND
Routing:
- net Vdrive: track 0.00 -> 146.2 mm, vias 0 -> 4
- net +5V: track 0.00 -> 96.7 mm, vias 0 -> 5
- net GND: track 0.00 -> 90.1 mm, vias 0 -> 72
- net /Start Up/VAUX: track 0.00 -> 89.7 mm, vias 0 -> 2
- net /Vout: track 0.00 -> 78.1 mm, vias 0 -> 2
- net /P1_1: track 0.00 -> 73.8 mm
- net /GND_drive1: track 0.00 -> 64.0 mm, vias 0 -> 9
- net /OP1-: track 0.00 -> 61.3 mm, vias 0 -> 2
- net VDD: track 0.00 -> 60.5 mm
- net /Vdrive2: track 0.00 -> 55.5 mm
- net Net-(Q2-B): track 0.00 -> 54.7 mm
- net /GND_drive2: track 0.00 -> 54.5 mm, vias 0 -> 9
- net GND1: track 0.00 -> 53.1 mm, vias 0 -> 14
- net /VFB: track 0.00 -> 52.4 mm
- net /Vdrive1: track 0.00 -> 46.2 mm
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- added copper zone on B.Cu, net /GND_drive1
- added copper zone on F.Cu, net /GND_drive1
- added copper zone on B.Cu, net /GND_drive2
- added copper zone on F.Cu, net /GND_drive2
- added copper zone on F.Cu, net /P1_1
- added copper zone on B.Cu, net GND
- added copper zone on F.Cu, net GND
- added copper zone on B.Cu, net GND1
- added copper zone on F.Cu, net GND1
- added copper zone on B.Cu, net GND2
- added copper zone on F.Cu, net GND2
- added copper zone on B.Cu, net GNDD
- added copper zone on F.Cu, net Net-(D10-K)
- added copper zone on F.Cu, net Net-(D11-K)
- added copper zone on F.Cu, net Net-(Q1-S)
- added copper zone on F.Cu, net Net-(R13-Pad2)
Other:
- outline, holes or cut-outs redrawn

Commit message: 初版PCB提交打样；
Parts:
- added TP14: GND, TestPoint:TestPoint_Keystone_5005-5009_Compact, F.Cu at (122.0, 54.3)
- added TP15: GND, TestPoint:TestPoint_Keystone_5005-5009_Compact, F.Cu at (92.9, 60.6)
- moved C1 2.49 mm to (92.2, 75.2), turned to -90 degrees
- moved J1 1.15 mm to (92.8, 56.4), turned to -90 degrees
- moved TP9 0.96 mm to (100.9, 84.2)
- moved R5 0.95 mm to (94.7, 74.4)
- moved Rost1 0.95 mm to (94.7, 72.9)
- moved TP8 0.47 mm to (101.0, 75.9)
- moved D11 0.21 mm to (108.5, 141.8)
Routing:
- net /ICSPCLK: track 4.26 -> 13.5 mm
- net /ICSPDAT: track 4.26 -> 9.79 mm
- net /MCLR: track 23.1 -> 27.7 mm
- net /OP1-: track 61.3 -> 57.5 mm
- net +5V: track 96.7 -> 93.0 mm
- net GND: track 90.1 -> 93.4 mm, vias 72 -> 74
- net /Isense: track 7.83 -> 6.53 mm
- net Net-(U1-RA2): track 10.5 -> 11.0 mm
- net /Drain: vias 0 -> 25
- net GNDD: vias 10 -> 9
- added copper zone on B.Cu, net /Drain
Other:
- outline, holes or cut-outs redrawn
- board text added: "+"
- board text added: "-"
- board text added: "BODE"
- board text added: "CS+"
- board text added: "Drain"
- board text added: "FunMod Design FlyBack"
- board text added: "GND"
- board text added: "GND1"
- board text added: "GND_drive1"
- board text added: "GND_drive2"
- board text added: "IN+"
- board text added: "IN-"
- board text added: "NEG"
- board text added: "P1+"
- board text added: "POS"
- board text added: "REF"
- board text added: "VFB"
- board text added: "Vdrive1"
- board text added: "Vdrive2"
- board text added: "Vout"
