File: FlyBack_pic16f1769.kicad_sch (KiCad schematic)
At the start: 108 parts, among them J1 ICSP, Q1 IPD50R380CE, T1 Transformer_PQ2020A_6+8, U1 PIC16F1769-I/P, U2 MCP1416

Commit message: 完善启动电路；
Parts:
- removed C35: 220p, Capacitor_SMD:C_1206_3216Metric_Pad1.33x1.80mm_HandSolder, symbol Device:C
- removed C36, C37, C38, C65: 10u, Capacitor_SMD:C_1206_3216Metric_Pad1.33x1.80mm_HandSolder, symbol Device:C
- removed C39: 100n, Capacitor_SMD:C_0603_1608Metric_Pad1.08x0.95mm_HandSolder, symbol Device:C
- removed C40: 10u, Capacitor_SMD:CP_Elec_10x12.5, symbol Device:C_Polarized
- removed D6: D, Diode_SMD:D_SMB_Handsoldering, symbol Device:D
- removed D9: Z1SMAxxx, Diode_SMD:D_SMA, symbol Diode:Z1SMAxxx
- removed R31, R32: 100, Resistor_SMD:R_1206_3216Metric_Pad1.30x1.75mm_HandSolder, symbol Device:R_Small_US
- removed R33, R34: 10k, Resistor_SMD:R_1206_3216Metric_Pad1.30x1.75mm_HandSolder, symbol Device:R_Small_US
- removed R53, R54, R55: 2k, Resistor_SMD:R_1206_3216Metric_Pad1.30x1.75mm_HandSolder, symbol Device:R_Small_US
- added CN1: 640445-3, kicad_api_lib:640445-3, symbol 640445-3:KF237-10.16-3P
- added CN2, CN5: 640445-2, kicad_api_lib:640445-2, symbol 640445-2:CH3.96-2A
- added TP10: Drain, TestPoint:TestPoint_Keystone_5005-5009_Compact, symbol Connector:TestPoint
- added TP8: Isense, TestPoint:TestPoint_Keystone_5005-5009_Compact, symbol Connector:TestPoint
- added TP9: GND, TestPoint:TestPoint_Keystone_5005-5009_Compact, symbol Connector:TestPoint
Connections:
- net Drain: now also TP10.1
- net GND: now also C43.2, C44.1, C45.1, C46.1, C47.1, R35.1, R36.1, T1.6, CN1.3, TP9.1
- net Vout: now also CN2.1
- net GND1: now reaches C13.1, C14.1, C15.1, C8.1, C9.2, R17.1, R18.1, T1.8
- net GND1: now also CN2.2
- net Vdrive1: now reaches C12.2, C16.2, C17.2, C18.2, C19.1, D3.1 (K), R19.2, R20.2, R21.2, R22.2
- net GND_drive1: now reaches C12.1, C16.1, C17.1, C18.1, C19.2, R21.1, R22.1, T1.10
- net at C29.1, C30.1, C31.1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: now also CN5.2
- net at C29.2, C30.2, C31.2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: now also CN5.1
- net GND_drive2: now reaches C22.1, C23.1, C24.1, C25.1, C26.2, R25.1, R26.1, T1.12
- net at C5.2, Q1.3 (S), R3.1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: now also TP8.1
- net Vdrive2: now reaches C22.2, C23.2, C24.2, C25.2, C26.1, D4.1 (K), R23.2, R24.2, R25.2, R26.2
- net Start Up/VAUX: now reaches R48.2
- net Vin renamed INPUT
- net INPUT: now also CN1.1
- no-connect marks 3 -> 7
Other:
- added sheet Driver (Driver.kicad_sch)
- added sheet Start Up (Start Up.kicad_sch)
- moved on the sheet: C61, C62, C63, C64, C66, D8, R17, R18, R29, R30, R35, R36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

Commit message: 初版布局连线；
Parts:
- removed C19, C26, C43: 10u, Capacitor_SMD:CP_Elec_10x12.5, symbol Device:C_Polarized
- added TP11: GND, TestPoint:TestPoint_Keystone_5005-5009_Compact, symbol Connector:TestPoint
- added TP13: Gate, TestPoint:TestPoint_Keystone_5005-5009_Compact, symbol Connector:TestPoint
Connections:
- net GND1: now also T1.14, TP11.1; no longer T1.8
- net GND2: now reaches C29.1, C30.1, C31.1, C32.1, C33.2, CN5.2, R29.1, R30.1
- net GND2: now also T1.8; no longer T1.14
- net at C28.1, D5.2 (A): now also T1.7; no longer T1.13
- net at C6.1, D1.2 (A): now also T1.13; no longer T1.7
- net at Q1.1 (G), R1.2, R2.2: now also TP13.1
Other:
- added sheet USB (USB.kicad_sch)
- sheet Start Up ports: added 5V_LDO, OP1-, OP1o/Ramp; removed none

Commit message: 初版PCB提交打样；
Parts:
- added TP14, TP15: GND, TestPoint:TestPoint_Keystone_5005-5009_Compact, symbol Connector:TestPoint
Connections:
- net GND: now also TP14.1, TP15.1
Changed lines of the file:
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@@
 	)
 	(junction
+		(at 57.15 33.02)
+		(diameter 0)
+		(color 0 0 0 0)
+	)
+	(junction
 		(at 146.05 153.67)
 		(diameter 0)
@@
 	)
 	(junction
+		(at 31.75 148.59)
+		(diameter 0)
+		(color 0 0 0 0)
+	)
+	(junction
 		(at 68.58 19.05)
 		(diameter 0)
@@
 	(wire
 		(pts
+			(xy 31.75 148.59) (xy 31.75 147.32)
+		)
+		(stroke
+			(width 0)
+			(type default)
+		)
+	)
+	(wire
+		(pts
 			(xy 176.53 36.83) (xy 176.53 72.39)
 		)
@@
 	(wire
 		(pts
-			(xy 31.75 149.86) (xy 31.75 147.32)
+			(xy 31.75 149.86) (xy 31.75 148.59)
 		)
 		(stroke
@@
 	(wire
 		(pts
-			(xy 48.26 33.02) (xy 68.58 33.02)
+			(xy 48.26 33.02) (xy 57.15 33.02)
 		)
 		(stroke
@@
 	(wire
 		(pts
+			(xy 57.15 33.02) (xy 68.58 33.02)
+		)
+		(stroke
+			(width 0)
+			(type default)
+		)
+	)
+	(wire
+		(pts
 			(xy 204.47 67.31) (xy 204.47 72.39)
 		)
@@
 	)
 	(symbol
+		(lib_id "Connector:TestPoint")
+		(at 31.75 148.59 90)
+		(unit 1)
+		(body_style 1)
+		(exclude_from_sim no)
+		(in_bom yes)
+		(on_board yes)
+		(in_pos_files yes)
+		(dnp no)
+		(fields_autoplaced yes)
+		(property "Reference" "TP15"
+			(at 28.448 143.51 90)
+			(show_name no)
+			(do_not_autoplace no)
+			(effects
+				(font
+					(size 1.27 1.27)
+				)
+			)
+		)
+		(property "Value" "GND"
+			(at 28.448 146.05 90)
+			(show_name no)
+			(do_not_autoplace no)
+			(effects
+				(font
+					(size 1.27 1.27)
+				)
+			)
+		)
+		(property "Footprint" "TestPoint:TestPoint_Keystone_5005-5009_Compact"
+			(at 31.75 143.51 0)
+			(hide yes)
+			(show_name no)
+			(do_not_autoplace no)
+			(effects
+				(font
+					(size 1.27 1.27)
+				)
+			)
+		)
+		(property "Datasheet" ""
+			(at 31.75 143.51 0)
+			(hide yes)
+			(show_name no)
+			(do_not_autoplace no)
+			(effects
+				(font
+					(size 1.27 1.27)
+				)
+			)
+		)
+		(property "Description" "test point"
+			(at 31.75 148.59 0)
+			(hide yes)
+			(show_name no)
+			(do_not_autoplace no)
+			(effects
+				(font
+					(size 1.27 1.27)
+				)
+			)
+		)
+		(pin "1"
+		)
+		(instances
+			(project "FlyBack_pic16f1769"
+				(path "/85fd1e61-7f7c-4adf-9ad3-eb5962af39d5"
+					(reference "TP15")
+					(unit 1)
+				)
+			)
+		)
+	)
+	(symbol
 		(lib_id "Device:C")
 		(at 224.79 29.21 180)
@@
 					(unit 1)
 				)
+			)
+		)
+	)
+	(symbol
+		(lib_id "Connector:TestPoint")
+		(at 57.15 33.02 180)
+		(unit 1)
+		(body_style 1)
+		(exclude_from_sim no)
+		(in_bom yes)
+		(on_board yes)
+		(in_pos_files yes)
+		(dnp no)
+		(fields_autoplaced yes)
+		(property "Reference" "TP14"
+			(at 59.69 35.0519 0)
+			(show_name no)
+			(do_not_autoplace no)
+			(effects
+				(font
+					(size 1.27 1.27)
+				)
+				(justify right)
+			)
+		)
+		(property "Value" "GND"
+			(at 59.69 37.5919 0)
+			(show_name no)
+			(do_not_autoplace no)
+			(effects
+				(font
+					(size 1.27 1.27)
+				)
+				(justify right)
+			)
+		)
+		(property "Footprint" "TestPoint:TestPoint_Keystone_5005-5009_Compact"
+			(at 52.07 33.02 0)
+			(hide yes)
+			(show_name no)
+			(do_not_autoplace no)
+			(effects
+				(font
+					(size 1.27 1.27)
+				)
+			)
+		)
+		(property "Datasheet" ""
+			(at 52.07 33.02 0)
+			(hide yes)
+			(show_name no)
+			(do_not_autoplace no)
+			(effects
+				(font
+					(size 1.27 1.27)
+				)
+			)
+		)
+		(property "Description" "test point"
+			(at 57.15 33.02 0)
+			(hide yes)
+			(show_name no)
+			(do_not_autoplace no)
+			(effects
+				(font
+					(size 1.27 1.27)
+				)
+			)
+		)
+		(pin "1"
+		)
+		(instances
+			(project "FlyBack_pic16f1769"
+				(path "/85fd1e61-7f7c-4adf-9ad3-eb5962af39d5"
+					(reference "TP14")
+					(unit 1)
+				)
